Commit message: fix: correct URDF structure for Gazebo simulation

File: models/arm_4r_physics.urdf (robot description, URDF)
Before this commit: robot robot_arm_4r, 7 links, 6 joints
Links:
- link base_rotation: mass None -> 0.15; geometry collision cylinder length=0.10 radius=0.035; visual cylinder length=0.10 radius=0.035
- link forearm: mass None -> 0.08; geometry collision box size=0.15 0.03 0.03; visual box size=0.15 0.03 0.03
- link wrist: mass None -> 0.05; geometry collision box size=0.06 0.025 0.025; visual box size=0.06 0.025 0.025
